File: hal9k-backlight/hal9k-backlight.sch (KiCad schematic (older format))
At the start: 14 parts, among them J1 +, J2 GND, J3 Din, J4 Dout

Commit message: backlight update
Parts:
- J1, J2, J3, J4: footprint Connector_PinSocket_2.00mm:PinSocket_1x01_P2.00mm_Vertical -> Connector_PinHeader_2.00mm:PinHeader_1x01_P2.00mm_Vertical
Changed lines of the file:
@@
 F 0 "J3" H 1170 1475 50  0000 C CNN
 F 1 "Din" H 1170 1566 50  0000 C CNN
-F 2 "Connector_PinSocket_2.00mm:PinSocket_1x01_P2.00mm_Vertical" H 1250 1700 50  0001 C CNN
+F 2 "Connector_PinHeader_2.00mm:PinHeader_1x01_P2.00mm_Vertical" H 1250 1700 50  0001 C CNN
 F 3 "~" H 1250 1700 50  0001 C CNN
 	1    1250 1700
@@
 F 0 "J2" V 1116 3712 50  0000 R CNN
 F 1 "GND" V 1025 3712 50  0000 R CNN
-F 2 "Connector_PinSocket_2.00mm:PinSocket_1x01_P2.00mm_Vertical" H 1150 3800 50  0001 C CNN
+F 2 "Connector_PinHeader_2.00mm:PinHeader_1x01_P2.00mm_Vertical" H 1150 3800 50  0001 C CNN
 F 3 "~" H 1150 3800 50  0001 C CNN
 	1    1150 3800
@@
 F 0 "J1" V 1023 3630 50  0000 L CNN
 F 1 "+" V 1114 3630 50  0000 L CNN
-F 2 "Connector_PinSocket_2.00mm:PinSocket_1x01_P2.00mm_Vertical" H 1150 3550 50  0001 C CNN
+F 2 "Connector_PinHeader_2.00mm:PinHeader_1x01_P2.00mm_Vertical" H 1150 3550 50  0001 C CNN
 F 3 "~" H 1150 3550 50  0001 C CNN
 	1    1150 3550
@@
 F 0 "J4" H 7180 1742 50  0000 L CNN
 F 1 "Dout" H 7180 1651 50  0000 L CNN
-F 2 "Connector_PinSocket_2.00mm:PinSocket_1x01_P2.00mm_Vertical" H 7100 1700 50  0001 C CNN
+F 2 "Connector_PinHeader_2.00mm:PinHeader_1x01_P2.00mm_Vertical" H 7100 1700 50  0001 C CNN
 F 3 "~" H 7100 1700 50  0001 C CNN
 	1    7100 1700
